Commit message: Renamed Joint position controllers.

File: simulation/gazebo-sim/shadow-bot/urdf/shadow.xacro (robot description, xacro)
@@ -37,4 +37,10 @@
               izz="${m*r*r/2}" />
   </macro>
+  <gazebo>
+    <plugin name="gazebo_ros_control" filename="libgazebo_ros_control.so">
+      <!-- <robotNamespace>/arboc</robotNamespace> -->
+      <!-- <robotSimType>gazebo_ros_control/DefaultRobotHWSim</robotSimType> -->
+    </plugin>
+  </gazebo>
  <link name="base_footprint">
     <inertial>
@@ -110,5 +116,5 @@
     <turnGravityOff>false</turnGravityOff>
   </gazebo>
-    <joint name="left_arm_joint" type="revolute">
+  <joint name="left_arm_joint" type="revolute">
     <parent link="base_link"/>
     <child link="left_arm"/>
@@ -121,8 +127,8 @@
     <type>transmission_interface/SimpleTransmission</type>
     <joint name="left_arm_joint">
-      <hardwareInterface>EffortJointInterface</hardwareInterface>
+      <hardwareInterface>hardware_interface/PositionJointInterface</hardwareInterface>
     </joint>
     <actuator name="left_arm_joint_motor">
-      <hardwareInterface>EffortJointInterface</hardwareInterface>
+      <hardwareInterface>hardware_interface/PositionJointInterface</hardwareInterface>
       <mechanicalReduction>500</mechanicalReduction>
     </actuator>
@@ -164,8 +170,8 @@
     <type>transmission_interface/SimpleTransmission</type>
     <joint name="right_arm_joint">
-      <hardwareInterface>EffortJointInterface</hardwareInterface>
+      <hardwareInterface>hardware_interface/PositionJointInterface</hardwareInterface>
     </joint>
     <actuator name="right_arm_joint_motor">
-      <hardwareInterface>EffortJointInterface</hardwareInterface>
+      <hardwareInterface>hardware_interface/PositionJointInterface</hardwareInterface>
       <mechanicalReduction>500</mechanicalReduction>
     </actuator>
@@ -186,6 +192,10 @@
       <alwaysOn>true</alwaysOn>
       <updateRate>100.0</updateRate>
-      <leftJoint>front_left_wheel_joint</leftJoint>
-      <rightJoint>front_right_wheel_joint</rightJoint>
+      <leftJoint name="front_left_wheel_joint">
+        <hardwareInterface>hardware_interface/PositionJointInterface</hardwareInterface>
+      </leftJoint>
+      <rightJoint name="front_right_wheel_joint">
+        <hardwareInterface>hardware_interface/PositionJointInterface</hardwareInterface>
+      </rightJoint>
       <wheelSeparation>${2*base_radius}</wheelSeparation>
       <wheelDiameter>${2*wheel_radius}</wheelDiameter>

File: simulation/gazebo-sim/shadow-bot/urdf/wheel.urdf.xacro (robot description, xacro)
@@ -57,7 +57,9 @@
     <transmission name="${fb}_${lr}_wheel_joint_trans">
       <type>transmission_interface/SimpleTransmission</type>
-      <joint name="${fb}_${lr}_wheel_joint" />
+      <joint name="${fb}_${lr}_wheel_joint">
+        <hardwareInterface>hardware_interface/PositionJointInterface</hardwareInterface>
+      </joint>
       <actuator name="${fb}_${lr}_wheel_joint_motor">
-        <hardwareInterface>EffortJointInterface</hardwareInterface>
+        <hardwareInterface>hardware_interface/PositionJointInterface</hardwareInterface>
         <mechanicalReduction>1</mechanicalReduction>
       </actuator>
@@ -105,7 +107,9 @@
     <transmission name="${fb}_${lr}_wheel_joint_trans">
       <type>transmission_interface/SimpleTransmission</type>
-      <joint name="${fb}_${lr}_wheel_joint" />
+      <joint name="${fb}_${lr}_wheel_joint">
+        <hardwareInterface>hardware_interface/PositionJointInterface</hardwareInterface>
+      </joint>
       <actuator name="${fb}_${lr}_wheel_joint_motor">
-        <hardwareInterface>EffortJointInterface</hardwareInterface>
+        <hardwareInterface>hardware_interface/PositionJointInterface</hardwareInterface>
         <mechanicalReduction>1</mechanicalReduction>
       </actuator>

Commit message: Fixed Moment of Inertia!

File: simulation/gazebo-sim/shadow-bot/urdf/shadow.xacro (robot description, xacro)
@@ -18,6 +18,4 @@
   <property name="DEG_TO_RAD" value="0.017453293" />
   <!-- body -->
-  <property name="base_height" value="0.02" />
-  <property name="base_radius" value="0.15" />
   <property name="base_mass" value="2.5" />
   <!-- arm -->
@@ -37,18 +35,14 @@
               izz="${m*r*r/2}" />
   </macro>
+  <macro name="box_inertia" params="m x y z">
+    <inertia  ixx="${m*(y*y+z*z)/12}" ixy = "0" ixz = "0"
+              iyy="${m*(x*x+z*z)/12}" iyz = "0"
+              izz="${m*(x*x+y*y)/12}" />
+  </macro>
   <gazebo>
     <plugin name="gazebo_ros_control" filename="libgazebo_ros_control.so">
-      <!-- <robotNamespace>/arboc</robotNamespace> -->
-      <!-- <robotSimType>gazebo_ros_control/DefaultRobotHWSim</robotSimType> -->
     </plugin>
   </gazebo>
  <link name="base_footprint">
-    <inertial>
-      <mass value="0.0001" />
-      <origin xyz="0 0 0" />
-      <inertia ixx="0.0001" ixy="0.0" ixz="0.0"
-          iyy="0.0001" iyz="0.0"
-          izz="0.0001" />
-    </inertial>
     <visual>
         <origin xyz="0 0 0" rpy="0 0 0" />
@@ -71,5 +65,5 @@
       <origin xyz="0 0 0" />
       <!--The 3x3 rotational inertia matrix. -->
-        <cylinder_inertia  m="${base_mass}" r="${base_radius}" h="${base_height}" />
+        <box_inertia  m="${base_mass}" x="0.262" y="0.150" z="0.06" />
     </inertial>
     <visual>
@@ -91,10 +85,10 @@
     <turnGravityOff>false</turnGravityOff>
   </gazebo>
-    <link name="left_arm">
+  <link name="left_arm">
     <inertial>
       <mass value="${arm_mass}" />
-      <origin xyz="0 0 0" />
+      <origin xyz="0.085 0 0" rpy="0 0 0 " />
       <!--The 3x3 rotational inertia matrix. -->
-        <cylinder_inertia  m="${base_mass}" r="${base_radius}" h="${base_height}" />
+        <box_inertia  m="${arm_mass}" x="0.170" y="0.015" z="0.025" />
     </inertial>
     <visual>
@@ -108,5 +102,5 @@
       <origin xyz="0.085 0 0" rpy="0 0 0 " />
       <geometry>
-          <box size="0.170 0.015 0.05" />
+          <box size="0.170 0.015 0.025" />
       </geometry>
     </collision>
@@ -121,6 +115,6 @@
     <origin xyz="0.0930 0.09 -0.0135" rpy="0 0 0" />
     <axis xyz="0 1 0"/>
-    <dynamics damping="1.0" friction="0.02"/>
-    <limit effort="7.0" lower="${-5*M_PI/12}" upper="${5*M_PI/12}" velocity="10.0"/>
+    <dynamics damping="0.0" friction="0.0"/>
+    <limit effort="1000.0" lower="${-5*M_PI/12}" upper="${5*M_PI/12}" velocity="1000.0"/>
   </joint>
   <transmission name="left_arm_joint_trans">
@@ -131,13 +125,13 @@
     <actuator name="left_arm_joint_motor">
       <hardwareInterface>hardware_interface/PositionJointInterface</hardwareInterface>
-      <mechanicalReduction>500</mechanicalReduction>
+      <mechanicalReduction>10</mechanicalReduction>
     </actuator>
   </transmission>
-    <link name="right_arm">
+  <link name="right_arm">
     <inertial>
       <mass value="${arm_mass}" />
-      <origin xyz="0 0 0" />
+      <origin xyz="0.085 0 0" rpy="0 0 0 " />
       <!--The 3x3 rotational inertia matrix. -->
-        <cylinder_inertia  m="${base_mass}" r="${base_radius}" h="${base_height}" />
+        <box_inertia  m="${arm_mass}" x="0.170" y="0.015" z="0.025" />
     </inertial>
     <visual>
@@ -151,5 +145,5 @@
       <origin xyz="0.085 0 0" rpy="0 0 0 " />
       <geometry>
-          <box size="0.170 0.015 0.05" />
+          <box size="0.170 0.015 0.025" />
       </geometry>
     </collision>
@@ -159,11 +153,11 @@
     <turnGravityOff>false</turnGravityOff>
   </gazebo>
-    <joint name="right_arm_joint" type="revolute">
+  <joint name="right_arm_joint" type="revolute">
     <parent link="base_link"/>
     <child link="right_arm"/>
     <origin xyz="0.0930 -0.09 -0.0135" rpy="0 0 0" />
     <axis xyz="0 1 0"/>
-    <dynamics damping="1.0" friction="0.02"/>
-    <limit effort="7.0" lower="${-5*M_PI/12}" upper="${5*M_PI/12}" velocity="10.0"/>
+    <dynamics damping="0.0" friction="0.0"/>
+    <limit effort="1000.0" lower="${-5*M_PI/12}" upper="${5*M_PI/12}" velocity="1000.0"/>
   </joint>
   <transmission name="right_arm_joint_trans">
@@ -174,5 +168,5 @@
     <actuator name="right_arm_joint_motor">
       <hardwareInterface>hardware_interface/PositionJointInterface</hardwareInterface>
-      <mechanicalReduction>500</mechanicalReduction>
+      <mechanicalReduction>10</mechanicalReduction>
     </actuator>
   </transmission>
@@ -194,8 +188,8 @@
       <leftJoint>front_left_wheel_joint</leftJoint>
       <rightJoint>front_right_wheel_joint</rightJoint>
-      <wheelSeparation>${2*base_radius}</wheelSeparation>
+      <wheelSeparation>0.150</wheelSeparation>
       <wheelDiameter>${2*wheel_radius}</wheelDiameter>
       <broadcastTF>1</broadcastTF>
-      <wheelTorque>30</wheelTorque>
+      <wheelTorque>40</wheelTorque>
       <wheelAcceleration>1.8</wheelAcceleration>
       <commandTopic>cmd_vel</commandTopic>

Commit message: Added new collada models to URDF.

File: simulation/gazebo-sim/shadow-bot/urdf/shadow.xacro (robot description, xacro)
@@ -20,5 +20,5 @@
   <property name="base_mass" value="2.5" />
   <!-- arm -->
-  <property name="arm_mass" value="0.15" />
+  <property name="arm_mass" value="1.0" />
   <!-- wheels -->
   <property name="wheel_mass" value="0.2" />
@@ -68,5 +68,5 @@
     </inertial>
     <visual>
-      <origin xyz="0.015 0 -0.03" rpy="0 0 0" />
+      <origin xyz="0.003 0 0.0065" rpy="0 0 ${M_PI/2}" />
       <geometry>
         <mesh filename="package://shadow-bot/meshes/dae/chassis.dae"/>
@@ -88,14 +88,14 @@
     <inertial>
       <mass value="${arm_mass}" />
-      <origin xyz="0.085 0 0" rpy="0 0 0 " />
+      <origin xyz="0.085 0 0" rpy="0 0 0" />
       <!--The 3x3 rotational inertia matrix. -->
         <box_inertia  m="${arm_mass}" x="0.170" y="0.015" z="0.025" />
     </inertial>
     <visual>
-      <origin xyz="-0.0775 -0.13115 0" rpy="0 0 0" />
-      <geometry>
-        <mesh filename="package://shadow-bot/meshes/dae/leftArmWheel.dae"/>
-      </geometry>
-      <material name="Black" />
+      <origin xyz="0.0625 0.02 0.0115" rpy="${-M_PI/5} 0 ${M_PI/2}" />
+      <geometry>
+        <mesh filename="package://shadow-bot/meshes/dae/left-arm.dae"/>
+      </geometry>
+      <material name="White" />
     </visual>
     <collision>
@@ -107,5 +107,5 @@
   </link>
   <gazebo reference="left_link">
-    <material>Gazebo/Black</material>
+    <material>Gazebo/White</material>
     <turnGravityOff>false</turnGravityOff>
   </gazebo>
@@ -131,14 +131,14 @@
     <inertial>
       <mass value="${arm_mass}" />
-      <origin xyz="0.085 0 0" rpy="0 0 0 " />
+      <origin xyz="0.085 0 0" rpy="0 0 0" />
       <!--The 3x3 rotational inertia matrix. -->
         <box_inertia  m="${arm_mass}" x="0.170" y="0.015" z="0.025" />
     </inertial>
     <visual>
-      <origin xyz="-0.0775 0.05115 0" rpy="0 0 0" />
-      <geometry>
-        <mesh filename="package://shadow-bot/meshes/dae/rightArmWheel.dae"/>
-      </geometry>
-      <material name="Black" />
+      <origin xyz="0.0625 -0.02 0.0115" rpy="${-M_PI/5} 0 ${M_PI/2}" />
+      <geometry>
+        <mesh filename="package://shadow-bot/meshes/dae/right-arm.dae"/>
+      </geometry>
+      <material name="White" />
     </visual>
     <collision>
@@ -150,5 +150,5 @@
   </link>
   <gazebo reference="right_link">
-    <material>Gazebo/Black</material>
+    <material>Gazebo/White</material>
     <turnGravityOff>false</turnGravityOff>
   </gazebo>
@@ -173,7 +173,7 @@
 <!-- Wheel Definitions -->
   <wheel fb="front" lr="right" parent="base_link" translateX="${base_x_origin_to_wheel_origin}" translateY="${base_y_origin_to_wheel_origin}" translateZ="${base_z_origin_to_wheel_origin}" flipY="1"/>
-  <wheel fb="front" lr="left" parent="base_link" translateX="${base_x_origin_to_wheel_origin}" translateY="-${base_y_origin_to_wheel_origin}" translateZ="${base_z_origin_to_wheel_origin}" flipY="1"/>
+  <wheel fb="front" lr="left" parent="base_link" translateX="${base_x_origin_to_wheel_origin}" translateY="-${base_y_origin_to_wheel_origin}" translateZ="${base_z_origin_to_wheel_origin}" flipY="-1"/>
   <arm_wheel fb="arm" lr="right" parent="right_arm" translateX="${arm_x_origin_to_wheel_origin}" translateY="${arm_y_origin_to_wheel_origin}" translateZ="${arm_z_origin_to_wheel_origin}" flipY="1"/>
-  <arm_wheel fb="arm" lr="left" parent="left_arm" translateX="${arm_x_origin_to_wheel_origin}" translateY="${-1 * arm_y_origin_to_wheel_origin}" translateZ="${arm_z_origin_to_wheel_origin}" flipY="1"/>
+  <arm_wheel fb="arm" lr="left" parent="left_arm" translateX="${arm_x_origin_to_wheel_origin}" translateY="${-1 * arm_y_origin_to_wheel_origin}" translateZ="${arm_z_origin_to_wheel_origin}" flipY="-1"/>
   <!-- Differential drive controller  -->
   <gazebo>
